File: Hardware/Spectacle_Button_Board.brd (EAGLE design)
At the start: 40 parts, among them J19 FTDI_DEVICE, U1 CY8C4146LQI-S422, U2 MIC5205-5V

Commit message: Laid out board
Parts:
- moved R5 246.6 mm to (-7.75, 38.7), turned to 180 degrees
- moved D2 236.2 mm to (-2.41, 38.7), turned to 270 degrees
- moved R6 232.1 mm to (-4.95, 16.0), turned to 90 degrees
- moved J18 229.7 mm to (5.08, 38.1), turned to 270 degrees
- moved SW2 223.3 mm to (-17.8, 24.4), turned to 180 degrees
- moved D3 223.2 mm to (-9.02, 16.0)
- moved SW1 222.0 mm to (-17.8, 27.9)
- moved JP1 220.8 mm to (-11.3, 45.1)
- moved R3 211.5 mm to (-11.2, 38.9), turned to 180 degrees
- moved R4 210.6 mm to (-15.0, 36.4), turned to 180 degrees
- moved D1 209.0 mm to (-18.0, 19.6)
- moved J19 206.2 mm to (-24.1, 27.9), turned to 270 degrees
- moved J17 199.2 mm to (5.08, 16.5), turned to 90 degrees
- moved C4 194.9 mm to (-5.21, 32.3), turned to 180 degrees
- moved C3 192.9 mm to (-5.21, 33.5), turned to 180 degrees
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Routing:
- net GND: track 0.00 -> 90.9 mm, vias 0 -> 5
- net 5V: track 0.00 -> 90.8 mm, vias 0 -> 8
- net XRES: track 0.00 -> 49.4 mm, vias 0 -> 1
- net VIN: track 0.00 -> 43.8 mm
- net SDA: track 0.00 -> 39.0 mm, vias 0 -> 2
- net SCL: track 0.00 -> 35.6 mm, vias 0 -> 2
- net IN_5: track 0.00 -> 34.3 mm, vias 0 -> 1
- net IN_1: track 0.00 -> 34.1 mm, vias 0 -> 1
- net IN_0: track 0.00 -> 33.8 mm, vias 0 -> 1
- net IN_2: track 0.00 -> 33.0 mm
- net IN_4: track 0.00 -> 32.2 mm, vias 0 -> 1
- net IN_6: track 0.00 -> 30.9 mm, vias 0 -> 1
- net IN_7: track 0.00 -> 27.7 mm, vias 0 -> 1
- net IN_3: track 0.00 -> 26.9 mm
- net SWD_DATA: track 0.00 -> 22.6 mm, vias 0 -> 1
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- added copper zone on layer 16, net GND
Other:
- board outline added: 34.3 x 62.2 mm
