File: Hardware/Spectacle_Button_Board.sch (EAGLE design)
At the start: 40 parts, among them J19 FTDI_DEVICE, U1 CY8C4146LQI-S422, U2 MIC5205-5V

Commit message: Laid out board
Other:
- note added: "C2 & C3 to be near U1G4.27"
- note added: "C4 to be near U1G4.25"
- note removed: "C2 & C3 to be near U1.27"
- note removed: "C4 to be near U1.25"
Changed lines of the file:
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@@
 <?xml version="1.0" encoding="utf-8"?>
 <!DOCTYPE eagle SYSTEM "eagle.dtd">
-<eagle version="7.5.0">
+<eagle version="7.2.0">
 <drawing>
 <settings>
@@
 hole headers</text>
 <text x="73.66" y="172.72" size="0.6096" layer="97">C2 &amp; C3 to be
-near U1.27</text>
+near U1G4.27</text>
 <text x="96.52" y="172.72" size="0.6096" layer="97">C4 to be
-near U1.25</text>
+near U1G4.25</text>
 </plain>
 <instances>
