File: Hardware/Spectacle_Motion_Board.sch (EAGLE design)
At the start: 48 parts, among them J10 AUDIO-JACK3, J3 USB-MICROB, J4 AUDIO-JACK3, U1 CY8C4146LQI-S422, U2 3.3V/150mA, U4 SN74LVC1G66, U5 SN74LVC1G66

Commit message: Added and fixed some product IDs
Parts:
- J11: device SparkFun-Connectors:M06NO_SILK_FEMALE_PTH -> SparkFun-Connectors:M06NO_SILK_NO_POP
- J5, J6, J7, J8, J9: PROD_ID (none) -> CONN-09692
Changed lines of the file:
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@@
 <layer number="19" name="Unrouted" color="6" fill="1" visible="no" active="no"/>
 <layer number="20" name="Dimension" color="15" fill="1" visible="no" active="no"/>
-<layer number="21" name="tPlace" color="7" fill="1" visible="no" active="no"/>
-<layer number="22" name="bPlace" color="7" fill="1" visible="no" active="no"/>
+<layer number="21" name="tPlace" color="16" fill="1" visible="no" active="no"/>
+<layer number="22" name="bPlace" color="14" fill="1" visible="no" active="no"/>
 <layer number="23" name="tOrigins" color="15" fill="1" visible="no" active="no"/>
 <layer number="24" name="bOrigins" color="15" fill="1" visible="no" active="no"/>
@@
 <layer number="27" name="tValues" color="7" fill="1" visible="no" active="no"/>
 <layer number="28" name="bValues" color="7" fill="1" visible="no" active="no"/>
-<layer number="29" name="tStop" color="15" fill="3" visible="no" active="no"/>
+<layer number="29" name="tStop" color="7" fill="3" visible="no" active="no"/>
 <layer number="30" name="bStop" color="7" fill="6" visible="no" active="no"/>
 <layer number="31" name="tCream" color="7" fill="4" visible="no" active="no"/>
@@
 <layer number="47" name="Measures" color="7" fill="1" visible="no" active="no"/>
 <layer number="48" name="Document" color="7" fill="1" visible="no" active="no"/>
-<layer number="49" name="Reference" color="13" fill="1" visible="no" active="no"/>
+<layer number="49" name="Reference" color="7" fill="1" visible="no" active="no"/>
 <layer number="50" name="dxf" color="7" fill="1" visible="no" active="no"/>
-<layer number="51" name="tDocu" color="14" fill="1" visible="no" active="no"/>
+<layer number="51" name="tDocu" color="6" fill="1" visible="no" active="no"/>
 <layer number="52" name="bDocu" color="7" fill="1" visible="no" active="no"/>
 <layer number="53" name="tGND_GNDA" color="7" fill="9" visible="no" active="no"/>
@@
 <part name="SUPPLY12" library="SparkFun-Aesthetics" deviceset="5V" device=""/>
 <part name="GND2" library="SparkFun-Aesthetics" deviceset="GND" device=""/>
-<part name="J5" library="SparkFun-Connectors" deviceset="M03" device="LOCK"/>
-<part name="J6" library="SparkFun-Connectors" deviceset="M03" device="LOCK"/>
-<part name="J7" library="SparkFun-Connectors" deviceset="M03" device="LOCK"/>
-<part name="J8" library="SparkFun-Connectors" deviceset="M03" device="LOCK"/>
-<part name="J9" library="SparkFun-Connectors" deviceset="M03" device="LOCK"/>
+<part name="J5" library="SparkFun-Connectors" deviceset="M03" device="LOCK">
+<attribute name="PROD_ID" value="CONN-09692"/>
+</part>
+<part name="J6" library="SparkFun-Connectors" deviceset="M03" device="LOCK">
+<attribute name="PROD_ID" value="CONN-09692"/>
+</part>
+<part name="J7" library="SparkFun-Connectors" deviceset="M03" device="LOCK">
+<attribute name="PROD_ID" value="CONN-09692"/>
+</part>
+<part name="J8" library="SparkFun-Connectors" deviceset="M03" device="LOCK">
+<attribute name="PROD_ID" value="CONN-09692"/>
+</part>
+<part name="J9" library="SparkFun-Connectors" deviceset="M03" device="LOCK">
+<attribute name="PROD_ID" value="CONN-09692"/>
+</part>
 <part name="SUPPLY13" library="SparkFun-Aesthetics" deviceset="5V" device=""/>
 <part name="SUPPLY14" library="SparkFun-Aesthetics" deviceset="5V" device=""/>
@@
 <part name="D5" library="SparkFun-DiscreteSemi" deviceset="DIODE-SCHOTTKY" device="-BAT20J" value="BAT20J"/>
 <part name="SUPPLY10" library="SparkFun-Aesthetics" deviceset="5V" device=""/>
-<part name="J11" library="SparkFun-Connectors" deviceset="M06" device="NO_SILK_FEMALE_PTH"/>
+<part name="J11" library="SparkFun-Connectors" deviceset="M06" device="NO_SILK_NO_POP"/>
 <part name="U4" library="SparkFun-AnalogIC" deviceset="SN74LVC1G66_SPST_AMUX" device="" value="SN74LVC1G66"/>
 <part name="U5" library="SparkFun-AnalogIC" deviceset="SN74LVC1G66_SPST_AMUX" device="" value="SN74LVC1G66"/>
@@
 <instance part="SUPPLY12" gate="G$1" x="104.14" y="73.66"/>
 <instance part="GND2" gate="1" x="88.9" y="55.88"/>
-<instance part="J5" gate="J$1" x="7.62" y="71.12"/>
-<instance part="J6" gate="J$1" x="7.62" y="55.88"/>
-<instance part="J7" gate="J$1" x="7.62" y="40.64"/>
-<instance part="J8" gate="J$1" x="38.1" y="71.12"/>
-<instance part="J9" gate="J$1" x="38.1" y="55.88"/>
+<instance part="J5" gate="J$1" x="7.62" y="71.12">
+<attribute name="PROD_ID" x="7.62" y="71.12" size="1.778" layer="96" display="off"/>
+</instance>
+<instance part="J6" gate="J$1" x="7.62" y="55.88">
+<attribute name="PROD_ID" x="7.62" y="55.88" size="1.778" layer="96" display="off"/>
+</instance>
+<instance part="J7" gate="J$1" x="7.62" y="40.64">
+<attribute name="PROD_ID" x="7.62" y="40.64" size="1.778" layer="96" display="off"/>
+</instance>
+<instance part="J8" gate="J$1" x="38.1" y="71.12">
+<attribute name="PROD_ID" x="38.1" y="71.12" size="1.778" layer="96" display="off"/>
+</instance>
+<instance part="J9" gate="J$1" x="38.1" y="55.88">
+<attribute name="PROD_ID" x="38.1" y="55.88" size="1.778" layer="96" display="off"/>
+</instance>
 <instance part="SUPPLY13" gate="G$1" x="20.32" y="78.74"/>
 <instance part="SUPPLY14" gate="G$1" x="50.8" y="78.74"/>

Commit message: Touchups for v10
Parts:
- J10, J4: value AUDIO-JACK3 -> TRRS_3.5mm; device SparkFun-Connectors:AUDIO-JACK3 -> SparkFun-Connectors:AUDIO_JACK_TRRSSMD_RA
Other:
- note added: "10"
- note removed: "03"
Changed lines of the file:
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@@
 <?xml version="1.0" encoding="utf-8"?>
 <!DOCTYPE eagle SYSTEM "eagle.dtd">
-<eagle version="7.6.0">
+<eagle version="7.7.0">
 <drawing>
 <settings>
@@
 <layer number="255" name="routoute" color="7" fill="1" visible="yes" active="yes"/>
 </layers>
-<schematic xreflabel="%F%N/%S" xrefpart="1_/%S.%C%R">
+<schematic xreflabel="%F%N/%S" xrefpart="/%S.%C%R">
 <attributes>
 </attributes>
@@
 <part name="SUPPLY9" library="SparkFun-Aesthetics" deviceset="3.3V" device=""/>
 <part name="SUPPLY11" library="SparkFun-Aesthetics" deviceset="3.3V" device=""/>
-<part name="J4" library="SparkFun-Connectors" deviceset="AUDIO-JACK3" device="">
+<part name="J4" library="SparkFun-Connectors" deviceset="AUDIO_JACK_TRRS" device="SMD_RA" value="TRRS_3.5mm">
 <attribute name="PROD_ID" value="CONN-10676"/>
 </part>
@@
 <part name="LOGO1" library="SparkFun-Aesthetics" deviceset="OSHW-LOGO" device="S"/>
 <part name="LOGO2" library="SparkFun-Aesthetics" deviceset="SFE_LOGO_NAME_FLAME" device=".1_INCH"/>
-<part name="J10" library="SparkFun-Connectors" deviceset="AUDIO-JACK3" device="">
+<part name="J10" library="SparkFun-Connectors" deviceset="AUDIO_JACK_TRRS" device="SMD_RA" value="TRRS_3.5mm">
 <attribute name="PROD_ID" value="CONN-10676"/>
 </part>
@@
 <wire x1="66.04" y1="86.36" x2="0" y2="86.36" width="0.3048" layer="97" style="longdash"/>
 <text x="165.1" y="7.62" size="3.81" layer="94" font="vector">Mike Hord</text>
-<text x="239.268" y="6.604" size="3.81" layer="94" font="vector">03</text>
+<text x="239.268" y="6.604" size="3.81" layer="94" font="vector">10</text>
 <wire x1="106.68" y1="114.3" x2="248.92" y2="114.3" width="0.3048" layer="97" style="longdash"/>
 <text x="109.22" y="116.84" size="3.81" layer="97" font="vector">MCU</text>
@@
 <instance part="LOGO1" gate="G$1" x="81.28" y="10.16"/>
 <instance part="LOGO2" gate="G$1" x="88.9" y="0"/>
-<instance part="J10" gate="G$1" x="190.5" y="53.34" rot="MR180">
+<instance part="J10" gate="G$1" x="190.5" y="53.34" smashed="yes" rot="MR180">
 <attribute name="PROD_ID" x="190.5" y="53.34" size="1.778" layer="96" rot="MR180" display="off"/>
+<attribute name="NAME" x="185.42" y="47.752" size="1.778" layer="95" font="vector" rot="MR180"/>
+<attribute name="VALUE" x="184.15" y="60.96" size="1.778" layer="96" font="vector" rot="MR180"/>
 </instance>
 <instance part="GND16" gate="1" x="198.12" y="43.18"/>
